File: lichtenstein_onion.brd (EAGLE design)
At the start: 73.9 x 54.2 mm, 48 parts, among them IC1 LM2852Y-3V3, J1 MAGJACK, U1 ONION-OMEGA2

Commit message: Got rid of resistor networks on lichtenstein board
Parts:
- removed RN1, RN2, RN3: 10k, resistor-net:CTS742C083
- added R14, R15, R16, R17, R18, R19, R20, R21, R22, R23, R24, R25: 10k, rcl:M0805
- IC2: value (none) -> MCP23017
Connections:
- net +3V3: now also R14.1, R15.1, R16.1, R17.1, R18.2, R19.2, R20.2, R21.2, R22.2, R23.2, R24.2, R25.2; no longer RN1.5, RN1.6, RN1.7, RN1.8, RN2.5, RN2.6, RN2.7, RN2.8, RN3.5, RN3.6, RN3.7, RN3.8
- net INPUT0: now also R18.1; no longer RN2.1
- net INPUT1: now also R19.1; no longer RN2.2
- net INPUT2: now also R24.1; no longer RN2.3
- net INPUT3: now also R25.1; no longer RN2.4
- net INPUT4: now also R20.1; no longer RN3.4
- net INPUT5: now also R21.1; no longer RN3.3
- net INPUT6: now also R23.1; no longer RN3.2
- net INPUT7: now also R22.1; no longer RN3.1
- net TEST0: now also R17.2; no longer RN1.4
- net TEST1: now also R16.2; no longer RN1.3
- net TEST2: now also R15.2; no longer RN1.2
- net TEST3: now also R14.2; no longer RN1.1
Routing:
- net INPUT3: track 34.1 -> 22.7 mm
- net INPUT4: track 28.1 -> 21.0 mm
- net INPUT2: track 29.1 -> 23.1 mm
- net +3V3: track 209.7 -> 215.2 mm, vias 3 -> 4
- net TEST3: track 42.8 -> 39.8 mm
- net INPUT5: track 27.8 -> 25.1 mm
- net INPUT6: track 27.4 -> 24.9 mm
- net INPUT7: track 26.2 -> 24.0 mm
- net TEST0: track 33.8 -> 32.2 mm
- net TEST2: track 39.4 -> 37.9 mm
- net INPUT0: track 18.3 -> 19.6 mm
- net TEST1: track 36.0 -> 35.2 mm
Other:
- board text added: "Lichtenstein-Onion Rev 03"
- board text removed: "Lichtenstein-Onion Rev 02"
