File: lichtenstein_onion.brd (EAGLE design)
At the start: 73.9 x 54.2 mm, 58 parts, among them IC1 LM2852Y-3V3, IC2 MCP23017, J1 MAGJACK, U1 ONION-OMEGA2

Commit message: Cleaned up traces slightly for PWM board
Connections:
- new net !SPI_CS_1: U1.J2-6
Changed lines of the file:
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@@
 <wire x1="54.6354" y1="39.5986" x2="54.6608" y2="39.5986" width="0.1524" layer="1"/>
+</signal>
+<signal name="!SPI_CS_1">
+<contactref element="U1" pad="J2-6"/>
 </signal>
 </signals>
