File: differential_output_board.brd (EAGLE design)
At the start: 100 x 50 mm, 23 parts, among them IC1 ATA6563

Commit message: added holes to differential output board
Parts:
- added H1, H2, H3: MOUNT-HOLE2.8, holes:2,8
Routing:
- net CANH_3: track 20.1 -> 24.6 mm
- net OUT3_N: track 59.4 -> 57.9 mm
- net OUT3_P: track 58.5 -> 57.4 mm
- net CANL_2: track 52.7 -> 53.5 mm
- net CANL_1: track 20.1 -> 20.8 mm
Other:
- board text added: "CAN Out CAN Return"
- board text added: "Ch0 Ch1 Ch2 Ch3"
- board text added: "Ch4 Ch5 Ch6 Ch7"
- board text removed: "Ch0 Ch1 CAN Out CAN Return Ch2 Ch3 CAN Out CAN Return"
- board text removed: "Ch4 Ch5 CAN Out CAN Return Ch6 Ch7 CAN Out CAN Return"

Commit message: More tweaks to the differential output board
Parts:
- IC1: value ATA6563 -> TJA1057
Changed lines of the file:
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@@
 <attribute name="SPICEPREFIX" value="C" x="46.71" y="3.04" size="1.778" layer="27" rot="R180" display="off"/>
 </element>
-<element name="IC1" library="lichtenstein_onion" package="SOIC8" value="ATA6563" x="35.5" y="33.5" smashed="yes" rot="R180">
+<element name="IC1" library="lichtenstein_onion" package="SOIC8" value="TJA1057" x="35.5" y="33.5" smashed="yes" rot="R180">
+<attribute name="MOUSER" value="771-TJA1057GT/3J" x="35.5" y="33.5" size="1.778" layer="27" rot="R180" display="off"/>
 <attribute name="NAME" x="38.167" y="35.405" size="0.8128" layer="25" font="vector" ratio="10" rot="R270"/>
 </element>
