File: lichtenstein_pwm_v2.brd (EAGLE design)
At the start: 71.9 x 117 mm, 76 parts, among them IC1 MCP23017, IC2 74AHCT125SOIC14, IC3 MAX11647, IC5 LM75B, IC7 LD1117, J1 MAGJACK, U1 ONION-OMEGA2

Commit message: pwm board v2: rev 01 sent to pcb fab
Parts:
- moved C20 2.87 mm to (21.1, 45.7)
Routing:
- net CURRENT: track 8.44 -> 10.0 mm
- net +3V3: track 291.4 -> 290.6 mm
Changed lines of the file:
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@@
 <?xml version="1.0" encoding="utf-8"?>
 <!DOCTYPE eagle SYSTEM "eagle.dtd">
-<eagle version="9.2.2">
+<eagle version="9.2.1">
 <drawing>
 <settings>
@@
 <element name="R24" library="rcl" library_urn="urn:adsk.eagle:library:334" package="M0805" package3d_urn="urn:adsk.eagle:package:23556/1" value="330R" x="24.13" y="44.704" smashed="yes" rot="MR270">
 <attribute name="MOUSER" value="71-CRCW0805330RFKEAC" x="24.13" y="44.704" size="1.778" layer="28" rot="MR270" display="off"/>
-<attribute name="NAME" x="22.098" y="46.482" size="1.27" layer="26" rot="MR270"/>
+<attribute name="NAME" x="19.558" y="40.894" size="1.27" layer="26" rot="MR90"/>
 <attribute name="SPICEPREFIX" value="R" x="24.13" y="44.704" size="1.778" layer="28" rot="MR270" display="off"/>
 <attribute name="VALUE" x="26.67" y="45.974" size="1.27" layer="28" rot="MR270"/>
 </element>
-<element name="C20" library="rcl" library_urn="urn:adsk.eagle:library:334" package="C0805" package3d_urn="urn:adsk.eagle:package:23617/2" value="100nF" x="23.114" y="47.752" smashed="yes" rot="MR0">
-<attribute name="MOUSER" value="710-885012207072" x="23.114" y="47.752" size="1.778" layer="28" rot="MR0" display="off"/>
-<attribute name="NAME" x="22.86" y="49.022" size="1.27" layer="26" rot="MR0"/>
-<attribute name="SPICEPREFIX" value="C" x="23.114" y="47.752" size="1.778" layer="28" rot="MR0" display="off"/>
-<attribute name="VALUE" x="24.384" y="45.212" size="1.27" layer="28" rot="MR0"/>
+<element name="C20" library="rcl" library_urn="urn:adsk.eagle:library:334" package="C0805" package3d_urn="urn:adsk.eagle:package:23617/2" value="100nF" x="21.082" y="45.72" smashed="yes" rot="MR0">
+<attribute name="MOUSER" value="710-885012207072" x="21.082" y="45.72" size="1.778" layer="28" rot="MR0" display="off"/>
+<attribute name="NAME" x="19.05" y="42.672" size="1.27" layer="26" rot="MR0"/>
+<attribute name="SPICEPREFIX" value="C" x="21.082" y="45.72" size="1.778" layer="28" rot="MR0" display="off"/>
+<attribute name="VALUE" x="22.352" y="43.18" size="1.27" layer="28" rot="MR0"/>
 </element>
 <element name="SV3" library="con-lstb" library_urn="urn:adsk.eagle:library:162" package="MA04-1" package3d_urn="urn:adsk.eagle:package:8337/1" value="" x="66.04" y="76.962" smashed="yes" rot="R270">
@@
 <contactref element="C10" pad="2"/>
 <contactref element="R23" pad="1"/>
-<via x="20.574" y="47.752" extent="1-16" drill="0.3048"/>
+<via x="23.114" y="48.768" extent="1-16" drill="0.3048"/>
 <via x="20.066" y="64.516" extent="1-16" drill="0.3048"/>
 <via x="18.034" y="67.564" extent="1-16" drill="0.3048"/>
@@
 <via x="22.098" y="70.358" extent="1-16" drill="0.3048"/>
 <via x="24.892" y="55.88" extent="1-16" drill="0.3048"/>
-<via x="30.734" y="52.324" extent="1-16" drill="0.3048"/>
+<via x="32.766" y="53.086" extent="1-16" drill="0.3048"/>
 <via x="45.593" y="44.704" extent="1-16" drill="0.3048"/>
 <via x="45.593" y="41.148" extent="1-16" drill="0.3048"/>
@@
 <wire x1="31.242" y1="42.926" x2="31.242" y2="47.752" width="0.2032" layer="16"/>
 <wire x1="30.546" y1="42.23" x2="30.546" y2="40.64" width="0.2032" layer="16"/>
-<wire x1="20.894" y1="100.584" x2="20.894" y2="100.076" width="0.4064" layer="1"/>
 <wire x1="28.956" y1="92.964" x2="30.099" y2="91.821" width="0.3048" layer="1"/>
 <wire x1="28.956" y1="92.964" x2="21.336" y2="92.964" width="0.3048" layer="1"/>
@@
 <wire x1="16.002" y1="100.076" x2="13.462" y2="97.536" width="0.4064" layer="1"/>
 <wire x1="13.208" y1="70.612" x2="13.208" y2="61.976" width="0.4064" layer="1"/>
-<wire x1="41.148" y1="80.772" x2="39.116" y2="82.804" width="0.3048" layer="16"/>
-<wire x1="39.116" y1="82.804" x2="35.94795" y2="82.804" width="0.3048" layer="16"/>
-<wire x1="35.94795" y1="82.804" x2="35.65715" y2="82.5132" width="0.3048" layer="16"/>
 <wire x1="13.208" y1="70.612" x2="13.462" y2="70.866" width="0.4064" layer="1"/>
 <wire x1="13.462" y1="70.866" x2="13.462" y2="72.39" width="0.4064" layer="1"/>
@@
 <wire x1="21.59" y1="79.756" x2="21.59" y2="81.026" width="0.4064" layer="1"/>
 <wire x1="21.59" y1="81.026" x2="21.59" y2="83.058" width="0.4064" layer="1"/>
-<wire x1="23.0772" y1="82.5132" x2="21.59" y2="81.026" width="0.3048" layer="16"/>
+<wire x1="21.59" y1="81.026" x2="23.0772" y2="82.5132" width="0.3048" layer="16"/>
 <via x="21.59" y="81.026" extent="1-16" drill="0.35"/>
-<wire x1="35.65715" y1="82.5132" x2="23.0772" y2="82.5132" width="0.3048" layer="16"/>
 <wire x1="20.894" y1="100.076" x2="20.894" y2="101.412" width="0.4064" layer="1"/>
 <wire x1="20.894" y1="101.412" x2="21.844" y2="102.362" width="0.4064" layer="1"/>
@@
 <wire x1="42.098" y1="46.294" x2="43.688" y2="46.294" width="0.3048" layer="1"/>
 <wire x1="40.5666" y1="50.8734" x2="41.656" y2="49.784" width="0.3048" layer="1"/>
+<wire x1="39.4068" y1="82.5132" x2="41.148" y2="80.772" width="0.3048" layer="16"/>
+<wire x1="23.0772" y1="82.5132" x2="39.4068" y2="82.5132" width="0.3048" layer="16"/>
 </signal>
 <signal name="CONSOLE_RX">
@@
 <contactref element="IC5" pad="1"/>
 <contactref element="IC3" pad="6"/>
-<wire x1="35.26" y1="77.516" x2="35.26" y2="77.472" width="0.2032" layer="1"/>
 <wire x1="17.526" y1="92.268" x2="18.73" y2="92.268" width="0.2032" layer="1"/>
 <wire x1="20.701" y1="90.297" x2="20.701" y2="90.214" width="0.2032" layer="1"/>
@@
 <wire x1="35.26" y1="77.77" x2="35.26" y2="77.472" width="0.2032" layer="1"/>
 <wire x1="27.686" y1="86.36" x2="30.226" y2="86.36" width="0.2032" layer="1"/>
-<wire x1="26.289" y1="90.214" x2="26.416" y2="90.087" width="0.2032" layer="1"/>
 <wire x1="16.51" y1="83.012" x2="16.51" y2="84.836" width="0.2032" layer="1"/>
 <wire x1="16.51" y1="84.836" x2="17.526" y2="85.852" width="0.2032" layer="1"/>
 <wire x1="17.526" y1="85.852" x2="17.526" y2="92.268" width="0.2032" layer="1"/>
 <wire x1="20.701" y1="90.214" x2="20.701" y2="89.027" width="0.2032" layer="1"/>
-<wire x1="20.701" y1="89.027" x2="20.828" y2="88.9" width="0.2032" layer="1"/>
-<wire x1="26.289" y1="90.214" x2="26.289" y2="88.9" width="0.2032" layer="1"/>
-<wire x1="26.289" y1="88.9" x2="26.289" y2="87.757" width="0.2032" layer="1"/>
+<wire x1="20.701" y1="89.027" x2="21.082" y2="88.646" width="0.2032" layer="1"/>
+<wire x1="26.289" y1="90.214" x2="26.289" y2="88.646" width="0.2032" layer="1"/>
+<wire x1="26.289" y1="88.646" x2="26.289" y2="87.757" width="0.2032" layer="1"/>
 <wire x1="26.289" y1="87.757" x2="27.686" y2="86.36" width="0.2032" layer="1"/>
-<wire x1="20.828" y1="88.9" x2="26.289" y2="88.9" width="0.2032" layer="1"/>
+<wire x1="21.082" y1="88.646" x2="26.289" y2="88.646" width="0.2032" layer="1"/>
 </signal>
 <signal name="SPI_MISO">
@@
 <wire x1="44.45" y1="37.786" x2="44.45" y2="40.64" width="0.2032" layer="1"/>
 <wire x1="45.004" y1="41.194" x2="45.004" y2="71.074" width="0.2032" layer="1"/>
-<wire x1="44.45" y1="40.64" x2="45.004" y2="41.194" width="0.2032" layer="1"/>
+<wire x1="45.004" y1="41.194" x2="44.45" y2="40.64" width="0.2032" layer="1"/>
 <wire x1="45.004" y1="71.074" x2="36.83" y2="79.248" width="0.2032" layer="1"/>
 </signal>
@@
 <contactref element="R24" pad="1"/>
 <contactref element="C20" pad="1"/>
-<wire x1="24.13" y1="45.654" x2="24.064" y2="45.72" width="0.2032" layer="16"/>
-<wire x1="24.064" y1="45.72" x2="24.064" y2="47.752" width="0.2032" layer="16"/>
-<wire x1="24.892" y1="47.752" x2="24.064" y2="47.752" width="0.2032" layer="16"/>
-<wire x1="27.178" y1="50.038" x2="24.892" y2="47.752" width="0.2032" layer="16"/>
+<wire x1="22.032" y1="45.72" x2="24.064" y2="45.72" width="0.2032" layer="16"/>
+<wire x1="24.064" y1="45.72" x2="24.13" y2="45.654" width="0.2032" layer="16"/>
+<wire x1="27.178" y1="50.038" x2="24.13" y2="46.99" width="0.2032" layer="16"/>
+<wire x1="24.13" y1="46.99" x2="24.13" y2="45.654" width="0.2032" layer="16"/>
 </signal>
 <signal name="N$12">
